File: hw/pcb/uedaino.sch (KiCad schematic (older format))
At the start: 35 parts, among them IC1 ATMEGA328P-A, P1 CN_PWR, P2 CN_UART, P3 CN_HEADER1, P4 CN_I2C, P5 CN_HEADER2, P6 CN_ICSP, SW1 SW_PUSH, SW2 SW_PWSEL, U1 AP1117, Y1 16MHz

Commit message: Add PCB Design
Parts:
- removed D2: LED_+3V3, Diodes_SMD:D_0603, symbol Led_Small
- removed JP7, JP8, JP9: Jumper_NC_Small, Pin_Headers:Pin_Header_Straight_1x02, symbol Jumper_NC_Small
- removed P1: CN_PWR, Connect:BARREL_JACK, symbol CONN_01X02
- removed P2: CN_UART, Pin_Headers:Pin_Header_Straight_1x05, symbol CONN_01X05
- removed P3: CN_HEADER1, Pin_Headers:Pin_Header_Straight_1x15, symbol CONN_01X15
- removed P4: CN_I2C, Pin_Headers:Pin_Header_Straight_1x04, symbol CONN_01X04
- removed P5: CN_HEADER2, Pin_Headers:Pin_Header_Straight_1x15, symbol CONN_01X15
- removed P6: CN_ICSP, Pin_Headers:Pin_Header_Straight_2x03, symbol CONN_02X03
- removed R6: 4.7K, Resistors_SMD:R_0603_HandSoldering, symbol R_Small
- removed SW2: SW_PWSEL, Pin_Headers:Pin_Header_Straight_1x03, symbol SWITCH_INV
- added P1: USB_OTG, Connectors:USB_Micro-B_10103594-0001LF, symbol USB_OTG
- added P2: CN_POWER, Socket_Strips:Socket_Strip_Straight_1x08, symbol CONN_01X08
- added P3: CN_J1, Socket_Strips:Socket_Strip_Straight_1x06, symbol CONN_01X06
- added P4: CN_ICSP, Socket_Strips:Socket_Strip_Straight_2x03, symbol CONN_02X03
- added P5: CONN_01X10, Socket_Strips:Socket_Strip_Straight_1x10, symbol CONN_01X10
- added P6: CONN_01X08, Socket_Strips:Socket_Strip_Straight_1x08, symbol CONN_01X08
- added U2: WS2812B, UeduinoLib:WS2812B, symbol WS2812B
- JP1: value Jumper_NC_Small -> J_CAP1; footprint Pin_Headers:Pin_Header_Straight_1x02 -> UeduinoLib:JP_CAP
- JP2: value Jumper_NC_Small -> J_CAP2; footprint Pin_Headers:Pin_Header_Straight_1x02 -> UeduinoLib:JP_CAP
- JP3: value Jumper_NC_Small -> J_CAP3; footprint Pin_Headers:Pin_Header_Straight_1x02 -> UeduinoLib:JP_CAP
- JP4: value Jumper_NC_Small -> J_CAP4; footprint Pin_Headers:Pin_Header_Straight_1x02 -> UeduinoLib:JP_CAP
- JP5: value Jumper_NC_Small -> J_CAP5; footprint Pin_Headers:Pin_Header_Straight_1x02 -> UeduinoLib:JP_CAP
- JP6: value Jumper_NC_Small -> J_CAP6; footprint Pin_Headers:Pin_Header_Straight_1x02 -> UeduinoLib:JP_CAP
- R4: value 1K -> 3.3K
- R5: value 4.7K -> 3.3K
- Y1: footprint Crystals:Crystal_HC49-SD_SMD -> Crystals:Crystal_SMD_5032_2Pads
- renumbered C6 to C3, C7 to C4, C4 to C5, C5 to C6, C3 to C7, R3 to R1, R1 to R2, R2 to R3
Connections:
- net labels added: AREF, D11/MOSI, D12/MISO, D13/SCK, IOREF, Vin
- net labels removed: D11, D12, D13, MISO, MOSI, PWR_USB, SCK
- wire segments 156 -> 132
- no-connect marks 2 -> 7
Other:
- note added: "CPU"
- note removed: "I2C"
- note removed: "ICSP"
- note removed: "UART"
- note removed: "aitendo AKIT-DTR340MC"
- moved on the sheet: C1, C2, C3, C4, C7, D1, IC1, R1, R2, R3, SW1, Y1

Commit message: Fix error
Parts:
- P1: symbol USB_OTG -> USB_OTG-RESCUE-uedaino
Changed lines of the file:
@@
 EESchema Schematic File Version 2
+LIBS:uedaino-rescue
 LIBS:power
 LIBS:device
@@
 LIBS:contrib
 LIBS:valves
-LIBS:kobayashi-lib
 LIBS:uedaino-cache
 EELAYER 25 0
@@
 $EndComp
 $Comp
-L USB_OTG P1
+L USB_OTG-RESCUE-uedaino P1
 U 1 1 58732FF4
 P 1100 1300
